File: hdw/UV_Blaster/UV_Blaster.kicad_pcb (KiCad board)
At the start: 4 copper layers, 241 parts, among them J201 +12V IN, J601 PICKIT3, J801 USB_B_Mini, Q1101 BSS214NW, Q201 Si4946BEY, Q401 BSS214NW, Q402 ZXMS6004FFTA, Q601 BSS214NW, SW1101 Cap_Touch, SW601 MRST, U1001 74LVC1G06, U1002 74LVC1G06, U1003 74LVC1G06, U1004 74LVC1G06, U1101 LTC6900, U1102 TLV71333PDBV, U1103 74LVC1G08, U1104 AT42QT1010-TSHR, U1105 74LVC1G17, U1106 MCP9804, U1201 LP8545, U1401 INA219BxDCN, U1402 MCP9804, U1403 INA219BxDCN, U201 LTC4365DDB, U301 INA219BxDCN, U302 MCP9804, U401 TPS62130, U501 INA219BxDCN, U502 MCP9804, U503 INA219BxDCN, U701 PIC18F27K40T-I_ML, U801 TLV6700, U802 FT234XD, U803 TPD3S014DBVR, U901 TPS71550, U902 74LVC1G06, U903 74LVC1G06, U904 74LVC1G06, X701 ECS-327KE

Commit message: Arranged input power parts
Parts:
- C301, C302, C303, U301, U302: moved to B.Cu
- moved L801 79.0 mm to (314.5, 63.2)
- moved C803 79.0 mm to (318.0, 55.2)
- moved C805 79.0 mm to (305.4, 63.0)
- moved C807 79.0 mm to (321.0, 55.2)
- moved C808 79.0 mm to (316.3, 59.9)
- moved C809 79.0 mm to (318.0, 57.3)
- moved D801 79.0 mm to (323.0, 52.6)
- moved J801 79.0 mm to (306.9, 55.8)
- moved R801 79.0 mm to (320.0, 61.7)
- moved R804 79.0 mm to (321.8, 59.5)
- moved U801 79.0 mm to (314.0, 56.5)
- moved C801 79.0 mm to (323.0, 50.6)
- moved C802 79.0 mm to (308.5, 63.0)
- moved C804 79.0 mm to (311.5, 63.1)
- moved C806 79.0 mm to (302.4, 63.0)
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Other:
- board text added: "+12V"
- board text added: "+12VIN"
